File: components/interfaces/hermetica-debugging-interface/hermetica-debugging-interface.kicad_pcb (KiCad board)
At the start: 2 copper layers, 45.7 x 27.9 mm, 15 parts, among them J1 JANOS-STACK-DEBUG-V1, J10 Conn_01x01, J11 Conn_01x01, J12 Conn_01x01, J2 CONNECTOR-DEBUG-SPECIFIC-ARM, J3 Conn_01x01, J4 Conn_01x01, J5 Conn_01x01, J6 Conn_01x01, J7 Conn_01x01, J8 Conn_01x01, J9 Conn_01x01, SW1 CUI-TS04, SW2 CUI-TS04

Commit message: updated pcbs
Changed lines of the file:
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@@
+		)
+	)
+	(dimension
+		(type orthogonal)
+		(layer "Eco2.User")
+		(pts
+			(xy 36.83 -13.97) (xy 36.83 13.97)
+		)
+		(height 3.81)
+		(orientation 1)
+		(format
+			(prefix "")
+			(suffix "")
+			(units 3)
+			(units_format 0)
+			(precision 4)
+			(suppress_zeroes yes)
+		)
+		(style
+			(thickness 0.1)
+			(arrow_length 1.27)
+			(text_position_mode 0)
+			(arrow_direction outward)
+			(extension_height 0.58642)
+			(extension_offset 0.5)
+			(keep_text_aligned yes)
+		)
+		(gr_text "27.94"
+			(at 39.49 0 90)
+			(layer "Eco2.User")
+			(effects
+				(font
+					(size 1 1)
+					(thickness 0.15)
+				)
+			)
+		)
+	)
+	(dimension
+		(type orthogonal)
+		(layer "Eco2.User")
+		(pts
+			(xy -8.89 -13.97) (xy 36.83 -13.97)
+		)
+		(height -3.175)
+		(orientation 0)
+		(format
+			(prefix "")
+			(suffix "")
+			(units 3)
+			(units_format 0)
+			(precision 4)
+			(suppress_zeroes yes)
+		)
+		(style
+			(thickness 0.1)
+			(arrow_length 1.27)
+			(text_position_mode 0)
+			(arrow_direction outward)
+			(extension_height 0.58642)
+			(extension_offset 0.5)
+			(keep_text_aligned yes)
+		)
+		(gr_text "45.72"
+			(at 13.97 -18.295 0)
+			(layer "Eco2.User")
+			(effects
+				(font
+					(size 1 1)
+					(thickness 0.15)
+				)
+			)
 		)
 	)
@@
 	(segment
 		(start -3.556 -3.5)
-		(end 8.0129 -3.5)
+		(end 7.056 -3.5)
+		(width 0.2)
+		(layer "F.Cu")
+		(net 1)
+	)
+	(segment
+		(start 13.4029 -8.89)
+		(end 15.875 -8.89)
+		(width 0.2)
+		(layer "F.Cu")
+		(net 1)
+	)
+	(segment
+		(start 9.74505 -6.18905)
+		(end 10.70195 -6.18905)
+		(width 0.2)
+		(layer "F.Cu")
+		(net 1)
+	)
+	(segment
+		(start 10.70195 -6.18905)
+		(end 13.4029 -8.89)
 		(width 0.2)
 		(layer "F.Cu")
@@
 	)
 	(segment
-		(start 8.0129 -3.5)
-		(end 13.4029 -8.89)
+		(start 7.056 -3.5)
+		(end 9.74505 -6.18905)
 		(width 0.2)
 		(layer "F.Cu")
-		(net 1)
-	)
-	(segment
-		(start 13.4029 -8.89)
-		(end 15.875 -8.89)
-		(width 0.2)
-		(layer "F.Cu")
