File: components/interfaces/hermetica-debugging-interface/hermetica-debugging-interface.kicad_sch (KiCad schematic)
At the start: 15 parts, among them J1 JANOS-STACK-DEBUG-V1, J10 Conn_01x01, J11 Conn_01x01, J12 Conn_01x01, J2 CONNECTOR-DEBUG-SPECIFIC-ARM, J3 Conn_01x01, J4 Conn_01x01, J5 Conn_01x01, J6 Conn_01x01, J7 Conn_01x01, J8 Conn_01x01, J9 Conn_01x01, SW1 CUI-TS04, SW2 CUI-TS04

Commit message: updated pcbs
Changed lines of the file:
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@@
 		(on_board yes)
 		(dnp no)
-		(fields_autoplaced yes)
 		(property "Reference" "SW1"
-			(at 95.25 71.12 0)
+			(at 95.25 72.644 0)
 			(effects
 				(font
@@
 		(on_board yes)
 		(dnp no)
-		(fields_autoplaced yes)
 		(property "Reference" "SW2"
-			(at 95.25 85.09 0)
-			(effects
-				(font
+			(at 95.25 86.868 0)
+			(effects
+				(font
