File: components/stack-layers/hermetica-fcustack-pdb/backplane.kicad_sch (KiCad schematic)
At the start: 14 parts, among them J1 Conn_02x14_Odd_Even, U4 LM66100DCK, U5 LM66100DCK, U6 74AHC1G17GWH

Commit message: FCU V2 REV1
Parts:
- removed J1: Conn_02x14_Odd_Even, Connector_PinSocket_2.54mm:PinSocket_2x14_P2.54mm_Vertical, symbol Connector_Generic:Conn_02x14_Odd_Even
- removed NT1: NetTie_2, NetTie:NetTie-2_THT_Pad0.3mm, symbol Device:NetTie_2
- added J3: Conn_02x50_Odd_Even, djStandard:SAMTEC-LSHM-150-XX.X-XX-DV-A-N, symbol DJ:Conn_02x50_Odd_Even
Connections:
- net +5V0: now also J3.89, J3.90, J3.91, J3.92
- net +5V0_CAN: now also J3.81, J3.82, J3.83, J3.84
- net BP_5V_RAIL_OK: now also J3.29 (Pin_29), J3.30 (Pin_30)
- net BP_ARMED: now also J3.21 (Pin_21), J3.22 (Pin_22)
- net BP_CAN1_H: now also J3.5 (Pin_5), J3.6 (Pin_6)
- net BP_CAN1_L: now also J3.1 (Pin_1), J3.2 (Pin_2)
- net BP_CAN2_H: now also J3.13 (Pin_13), J3.14 (Pin_14)
- net BP_CAN2_L: now also J3.10 (Pin_10), J3.9 (Pin_9)
- net BP_SAFE: now also J3.25 (Pin_25), J3.26 (Pin_26)
- net BP_SYNC: now also J3.17 (Pin_17), J3.18 (Pin_18)
- net BP_VBAT_2A: now also J3.100, J3.97, J3.98, J3.99
- net GND: now also J3.11 (Pin_11), J3.12 (Pin_12), J3.15 (Pin_15), J3.16 (Pin_16), J3.19 (Pin_19), J3.20 (Pin_20), J3.23 (Pin_23), J3.24 (Pin_24), J3.27 (Pin_27), J3.28 (Pin_28), J3.3 (Pin_3), J3.31 (Pin_31), J3.32 (Pin_32), J3.33 (Pin_33), J3.34 (Pin_34), J3.35 (Pin_35), J3.36 (Pin_36), J3.37 (Pin_37), J3.38 (Pin_38), J3.39 (Pin_39), J3.4 (Pin_4), J3.40 (Pin_40), J3.41 (Pin_41), J3.42 (Pin_42), J3.43 (Pin_43), J3.44 (Pin_44), J3.45 (Pin_45), J3.46 (Pin_46), J3.47 (Pin_47), J3.48 (Pin_48), J3.49 (Pin_49), J3.50 (Pin_50), J3.51 (Pin_51), J3.52 (Pin_52), J3.53 (Pin_53), J3.54 (Pin_54), J3.55 (Pin_55), J3.56 (Pin_56), J3.57 (Pin_57), J3.58 (Pin_58), J3.59 (Pin_59), J3.60 (Pin_60), J3.61 (Pin_61), J3.62 (Pin_62), J3.63 (Pin_63), J3.64 (Pin_64), J3.65 (Pin_65), J3.66 (Pin_66), J3.67 (Pin_67), J3.68 (Pin_68), J3.69 (Pin_69), J3.7 (Pin_7), J3.70 (Pin_70), J3.71 (Pin_71), J3.72 (Pin_72), J3.73 (Pin_73), J3.74 (Pin_74), J3.77 (Pin_77), J3.78 (Pin_78), J3.79 (Pin_79), J3.8 (Pin_8), J3.80 (Pin_80), J3.85, J3.86, J3.87, J3.88, J3.93, J3.94, J3.95, J3.96
- no-connect marks 0 -> 1
