File: components/stack-layers/hermetica-fcustack-pdb/can.kicad_sch (KiCad schematic)
At the start: 22 parts, among them U18 PESD2CANFD24V-QCZ, U21 PESD2CANFD24V-QCZ

Commit message: FCU V2 REV1
Connections:
- net BP_CAN1_H: now also U18.1 (K1); no longer U18.2 (K2)
- net BP_CAN1_L: now also U18.2 (K2); no longer U18.1 (K1)
- net BP_CAN2_H: now also U21.1 (K1); no longer U21.2 (K2)
- net BP_CAN2_L: now also U21.2 (K2); no longer U21.1 (K1)
Changed lines of the file:
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@@
 	(global_label "BP_CAN1_H"
 		(shape bidirectional)
-		(at 45.72 45.72 180)
-		(fields_autoplaced yes)
-		(effects
-			(font
-				(size 1.27 1.27)
-			)
-			(justify right)
-		)
-		(property "Intersheetrefs" "${INTERSHEET_REFS}"
-			(at 30.9192 45.72 0)
+		(at 45.72 40.64 180)
+		(fields_autoplaced yes)
+		(effects
+			(font
+				(size 1.27 1.27)
+			)
+			(justify right)
+		)
+		(property "Intersheetrefs" "${INTERSHEET_REFS}"
+			(at 30.9192 40.64 0)
 			(effects
 				(font
@@
 	(global_label "BP_CAN2_L"
 		(shape bidirectional)
-		(at 48.26 110.49 180)
-		(fields_autoplaced yes)
-		(effects
-			(font
-				(size 1.27 1.27)
-			)
-			(justify right)
-		)
-		(property "Intersheetrefs" "${INTERSHEET_REFS}"
-			(at 33.7616 110.49 0)
+		(at 48.26 115.57 180)
+		(fields_autoplaced yes)
+		(effects
+			(font
+				(size 1.27 1.27)
+			)
+			(justify right)
+		)
+		(property "Intersheetrefs" "${INTERSHEET_REFS}"
+			(at 33.7616 115.57 0)
 			(effects
 				(font
@@
 	(global_label "BP_CAN2_H"
 		(shape bidirectional)
-		(at 48.26 115.57 180)
-		(fields_autoplaced yes)
-		(effects
-			(font
-				(size 1.27 1.27)
-			)
-			(justify right)
-		)
-		(property "Intersheetrefs" "${INTERSHEET_REFS}"
-			(at 33.4592 115.57 0)
+		(at 48.26 110.49 180)
+		(fields_autoplaced yes)
+		(effects
+			(font
+				(size 1.27 1.27)
+			)
+			(justify right)
+		)
+		(property "Intersheetrefs" "${INTERSHEET_REFS}"
+			(at 33.4592 110.49 0)
 			(effects
 				(font
@@
 	(global_label "BP_CAN1_L"
 		(shape bidirectional)
-		(at 45.72 40.64 180)
-		(fields_autoplaced yes)
-		(effects
-			(font
-				(size 1.27 1.27)
-			)
-			(justify right)
-		)
-		(property "Intersheetrefs" "${INTERSHEET_REFS}"
-			(at 31.2216 40.64 0)
-			(effects
-				(font
+		(at 45.72 45.72 180)
+		(fields_autoplaced yes)
+		(effects
+			(font
+				(size 1.27 1.27)
+			)
+			(justify right)
+		)
+		(property "Intersheetrefs" "${INTERSHEET_REFS}"
+			(at 31.2216 45.72 0)
+			(effects
+				(font
