File: components/stack-layers/hermetica-fcustack-pdb/hermetica-fcustack-pdb.kicad_pcb (KiCad board)
At the start: 4 copper layers, 70.5 x 50.8 mm, 143 parts, among them IC1 SN74LVC1G14-Q1, J1 Conn_02x14_Odd_Even, J2 JANOS-STACK-DEBUG-V1, Q1 NPN, Q4 NEXPERIA-BSS138-SOT-23-3, Q5 DDTC114EE-7-F, Q6 DIODESINC-MMBT4401-7-F-SOT-23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, U1 74AHC1G17GWH, U10 74AHC1G17GWH, U11 74AHC1G17GWH, U12 74AHC1G17GWH, U13 74AUC1G08, U14 74AHCT1G32, U15 74AHC1G17GWH, U16 74AHCT121A, U17 74AHC1G17GWH, U18 PESD2CANFD24V-QCZ, U2 74AHC1G17GWH, U21 PESD2CANFD24V-QCZ, U22 TPSM63603V5RDHR, U23 TPS22991BRAAR, U24 INA240A1D, U3 74AHC1G17GWH, U4 LM66100DCK, U5 LM66100DCK, U6 74AHC1G17GWH, U7 MB85RS1MT, U8 LP5912-3.3DRV, U9 LM66100DCK, Y1 ABRACON-ABM10AIG-48.000MHZ-4Z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

Commit message: FCU V2 REV1
Parts:
- removed H1, H10, H2, H3, H5, H7, H8, H9: MountingHole_Pad, djStandard:MountingHole_M2.5_AWG14_SmallPad
- removed J1: Conn_02x14_Odd_Even, Connector_PinSocket_2.54mm:PinSocket_2x14_P2.54mm_Vertical
- removed NT1, NT4: NetTie_2, NetTie:NetTie-2_THT_Pad0.3mm
- removed U24: INA240A1D, Package_SO:SOIC-8_3.9x4.9mm_P1.27mm
- added J3: Conn_02x50_Odd_Even, djStandard:SAMTEC-LSHM-150-XX.X-XX-DV-A-N, F.Cu at (-31.8, 0.00)
- added J4: JANOS-STACK-CAN, djStandard:SAMTEC-T1M-03-F-SH-L, F.Cu at (47.5, -27.7)
- added U25: INA238, Package_SO:VSSOP-10_3x3mm_P0.5mm, F.Cu at (50.2, 13.3)
- RS2: footprint djStandard:OHMITE-PCS-1206 -> djStandard:VISHAY-WSL27261L300FEA
- U18, U21: moved to B.Cu
- moved C13 88.1 mm to (0.38, -7.92), turned to 180 degrees
- moved C14 87.7 mm to (0.38, -12.5)
- moved Y1 85.8 mm to (0.38, -10.2), turned to 90 degrees
- moved R7 81.2 mm to (-10.9, -4.75), turned to -90 degrees
- moved D4 80.0 mm to (83.0, 52.3), turned to 0 degrees
- moved RS2 76.6 mm to (73.5, 48.2), turned to 0 degrees
- moved R11 74.5 mm to (-8.38, -20.2), turned to -90 degrees
- moved NT2 73.9 mm to (80.8, 34.9), turned to 0 degrees
- moved NT3 73.2 mm to (80.8, 36.5), turned to 0 degrees
- moved H4 64.0 mm to (65.2, 46.0)
- moved H6 60.8 mm to (65.2, 52.1)
- moved R19 54.7 mm to (-10.9, 10.9)
- moved R10 51.2 mm to (-7.37, -20.2), turned to -90 degrees
- moved R9 46.6 mm to (-10.2, -4.75), turned to -90 degrees
- moved MCU1 42.0 mm to (-8.13, -10.7), turned to 180 degrees
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Connections:
- D4 pad 1: /primary-power/BATTERY_2S_TO_8S -> /primary-power/INCOMING_2S_TO_8S+
- H6 pad 1: /primary-power/INCOMING_2S_TO_8S- -> GND
- J2 pad 3: /mcu/SWCLK -> GND
- J2 pad 4: /mcu/SWO -> /mcu/SWCLK
- J2 pad 5: /mcu/BOOT0 -> /mcu/SWO
- J2 pad 6: /mcu/RESET -> /mcu/BOOT0
- J2 pad 7: /mcu/USART3_TX -> /mcu/RESET
- J2 pad 8: /mcu/USART3_RX -> /mcu/USART3_TX
- J2 pad 9: GND -> /mcu/USART3_RX
- U18 pad 1: BP_CAN1_L -> BP_CAN1_H
- U18 pad 2: BP_CAN1_H -> BP_CAN1_L
- U21 pad 1: BP_CAN2_L -> BP_CAN2_H
- U21 pad 2: BP_CAN2_H -> BP_CAN2_L
Routing:
- net PRIMARY_POWER: track 138.9 -> 4.12 mm, vias 14 -> 12
- net GND: track 122.8 -> 0.00 mm, vias 11 -> 10
- net +5V0: track 65.6 -> 34.9 mm
- net /mcu/SWO: track 0.00 -> 28.4 mm, vias 0 -> 2
- net /mcu/SWCLK: track 0.00 -> 26.3 mm, vias 0 -> 2
- net /mcu/RESET: track 1.15 -> 26.1 mm, vias 1 -> 2
- net /mcu/BOOT0: track 1.95 -> 26.9 mm, vias 1 -> 2
- net /mcu/SWDIO: track 0.00 -> 22.5 mm, vias 0 -> 2
- net /mcu/USART3_TX: track 0.00 -> 20.2 mm, vias 0 -> 2
- net /mcu/USART3_RX: track 0.00 -> 18.1 mm, vias 0 -> 2
- net /mcu/OSC+: track 0.00 -> 7.85 mm
- net /mcu/OSC-: track 0.00 -> 5.48 mm
- net /mcu/LED_GREEN: track 0.00 -> 5.06 mm
- net /mcu/LED_RED: track 0.00 -> 4.86 mm
- net Net-(U19-RXD): track 0.00 -> 4.18 mm
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- added copper zone on F.Cu, net /backplane/BP_VBAT_2A
- removed copper zone on F.Cu, net /primary-power/INCOMING_2S_TO_8S+
Other:
- outline, holes or cut-outs redrawn
