File: components/stack-layers/hermetica-fcustack-pdb/hermetica-fcustack-pdb.kicad_sch (KiCad schematic)
At the start: 16 parts, among them U1 74AHC1G17GWH, U2 74AHC1G17GWH, U3 74AHC1G17GWH

Commit message: FCU V2 REV1
Changed lines of the file:
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@@
 	)
 	(sheet
-		(at 219.964 148.59)
+		(at 219.964 149.86)
 		(size 24.384 10.668)
 		(exclude_from_sim no)
@@
 		)
 		(property "Sheetname" "stack-power"
-			(at 219.964 147.8784 0)
+			(at 219.964 149.1484 0)
 			(effects
 				(font
@@
 		)
 		(property "Sheetfile" "stack-power.kicad_sch"
-			(at 219.964 159.8426 0)
+			(at 219.964 161.1126 0)
 			(effects
 				(font
