File: components/stack-layers/hermetica-fcustack-pdb/mcu.kicad_sch (KiCad schematic)
At the start: 23 parts, among them J2 JANOS-STACK-DEBUG-V1, J3 JANOS-STACK-DEBUG-V1, J4 JANOS-STACK-CAN, U7 MB85RS1MT, Y1 ABRACON-ABM10AIG-48.000MHZ-4Z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

Commit message: FCU V2 REV1
Parts:
- removed J3: JANOS-STACK-DEBUG-V1, djStandard:SAMTEC-T1M-10-F-SH-L, symbol DJ:JANOS-STACK-DEBUG-V1
Connections:
- net +3V3: now also J2.1 (VTARGET)
- net BOOT0: now also J2.6 (BOOT0)
- net GND: now also J2.10 (GND), J2.3 (nSERVICEPORT), J2.S1, J2.S2
- net RESET: now also J2.7 (~{RESET})
- net SWCLK: now also J2.4 (SWCLK)
- net SWDIO: now also J2.2 (SWDIO)
- net SWO: now also J2.5 (SWO)
- net USART3_RX: now also J2.9 (MCU_RX)
- net USART3_TX: now also J2.8 (MCU_TX)
Changed lines of the file:
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@@
 	)
 	(junction
+		(at 52.07 127)
+		(diameter 0)
+		(color 0 0 0 0)
+	)
+	(junction
 		(at 177.8 50.8)
 		(diameter 0)
@@
 	)
 	(junction
+		(at 52.07 121.92)
+		(diameter 0)
+		(color 0 0 0 0)
+	)
+	(junction
 		(at 137.16 53.34)
 		(diameter 0)
@@
 	)
 	(junction
+		(at 52.07 124.46)
+		(diameter 0)
+		(color 0 0 0 0)
+	)
+	(junction
 		(at 193.04 34.29)
 		(diameter 0)
@@
 	(wire
 		(pts
+			(xy 52.07 124.46) (xy 52.07 127)
+		)
+		(stroke
+			(width 0)
+			(type default)
+		)
+	)
+	(wire
+		(pts
 			(xy 180.34 50.8) (xy 182.88 50.8)
 		)
@@
 	(wire
 		(pts
-			(xy 41.91 121.92) (xy 41.91 129.54)
+			(xy 52.07 121.92) (xy 52.07 124.46)
 		)
 		(stroke
@@
 	(wire
 		(pts
-			(xy 22.86 119.38) (xy 35.56 119.38)
+			(xy 39.37 116.84) (xy 52.07 116.84)
 		)
 		(stroke
@@
 	(wire
 		(pts
-			(xy 22.86 114.3) (xy 35.56 114.3)
+			(xy 39.37 111.76) (xy 52.07 111.76)
 		)
 		(stroke
@@
 	(wire
 		(pts
-			(xy 22.86 116.84) (xy 35.56 116.84)
+			(xy 39.37 114.3) (xy 52.07 114.3)
+		)
+		(stroke
+			(width 0)
+			(type default)
+		)
+	)
+	(wire
+		(pts
+			(xy 52.07 127) (xy 52.07 129.54)
 		)
 		(stroke
@@
 	(wire
 		(pts
+			(xy 52.07 119.38) (xy 52.07 121.92)
+		)
+		(stroke
+			(width 0)
+			(type default)
+		)
+	)
+	(wire
+		(pts
 			(xy 238.76 99.06) (xy 238.76 104.14)
 		)
@@
 	(wire
 		(pts
-			(xy 22.86 109.22) (xy 35.56 109.22)
+			(xy 39.37 106.68) (xy 52.07 106.68)
 		)
 		(stroke
@@
 	(wire
 		(pts
-			(xy 22.86 111.76) (xy 35.56 111.76)
+			(xy 39.37 109.22) (xy 52.07 109.22)
 		)
 		(stroke
@@
 	(wire
 		(pts
-			(xy 22.86 104.14) (xy 35.56 104.14)
+			(xy 39.37 101.6) (xy 52.07 101.6)
 		)
 		(stroke
@@
 	(wire
 		(pts
-			(xy 22.86 106.68) (xy 35.56 106.68)
+			(xy 39.37 104.14) (xy 52.07 104.14)
 		)
 		(stroke
@@
 	)
 	(label "SWCLK"
-		(at 22.86 106.68 0)
+		(at 39.37 104.14 0)
 		(effects
 			(font
@@
 	)
 	(label "USART3_RX"
-		(at 22.86 119.38 0)
+		(at 39.37 116.84 0)
 		(effects
 			(font
@@
 	)
 	(label "SWDIO"
-		(at 22.86 104.14 0)
+		(at 39.37 101.6 0)
 		(effects
 			(font
@@
 	)
 	(label "RESET"
-		(at 22.86 114.3 0)
+		(at 39.37 111.76 0)
 		(effects
 			(font
@@
 	)
 	(label "BOOT0"
-		(at 22.86 111.76 0)
+		(at 39.37 109.22 0)
 		(effects
 			(font
@@
 	)
 	(label "SWO"
-		(at 22.86 109.22 0)
+		(at 39.37 106.68 0)
 		(effects
 			(font
@@
 	)
 	(label "USART3_TX"
-		(at 22.86 116.84 0)
+		(at 39.37 114.3 0)
 		(effects
 			(font
@@
 	(symbol
 		(lib_id "DJ:+3V3")
-		(at 41.91 101.6 0)
+		(at 52.07 99.06 0)
 		(unit 1)
 		(exclude_from_sim no)
@@
 		(fields_autoplaced yes)
 		(property "Reference" "#PWR038"
-			(at 41.91 105.41 0)
+			(at 52.07 102.87 0)
 			(effects
 				(font
@@
 		)
 		(property "Value" "+3V3"
-			(at 41.91 98.044 0)
+			(at 52.07 95.504 0)
 			(effects
 				(font
@@
 		)
 		(property "Footprint" ""
-			(at 41.91 101.6 0)
+			(at 52.07 99.06 0)
 			(effects
 				(font
@@
 		)
 		(property "Datasheet" ""
-			(at 41.91 101.6 0)
+			(at 52.07 99.06 0)
 			(effects
 				(font
@@
 		)
 		(property "Description" "Power - Power symbol creates a global label with name \"+3V3\""
-			(at 41.91 101.6 0)
+			(at 52.07 99.06 0)
 			(effects
 				(font
@@
 	(symbol
 		(lib_id "DJ:GND")
-		(at 41.91 129.54 0)
+		(at 52.07 129.54 0)
 		(unit 1)
 		(exclude_from_sim no)
@@
 		(fields_autoplaced yes)
 		(property "Reference" "#PWR041"
-			(at 41.91 135.89 0)
+			(at 52.07 135.89 0)
 			(effects
 				(font
@@
 		)
 		(property "Value" "GND"
-			(at 41.91 133.35 0)
+			(at 52.07 133.35 0)
 			(effects
 				(font
@@
 		)
 		(property "Footprint" ""
-			(at 41.91 129.54 0)
+			(at 52.07 129.54 0)
 			(effects
 				(font
@@
 		)
 		(property "Datasheet" ""
-			(at 41.91 129.54 0)
+			(at 52.07 129.54 0)
 			(effects
 				(font
@@
 		)
 		(property "Description" "Power symbol creates a global label with name \"GND\" , ground"
-			(at 41.91 129.54 0)
+			(at 52.07 129.54 0)
 			(effects
 				(font
@@
 					(unit 1)
 				)
-			)
-		)
-	)
-	(symbol
-		(lib_id "DJ:JANOS-STACK-DEBUG-V1")
-		(at -19.05 86.36 0)
-		(unit 1)
-		(exclude_from_sim no)
-		(in_bom yes)
-		(on_board yes)
-		(dnp no)
-		(fields_autoplaced yes)
-		(property "Reference" "J3"
-			(at -7.62 99.1869 0)
-			(effects
-				(font
-					(size 1.27 1.27)
-				)
-				(justify left)
-			)
-		)
-		(property "Value" "JANOS-STACK-DEBUG-V1"
-			(at 12.7 88.9 0)
-			(effects
-				(font
-					(size 1.27 1.27)
-				)
-				(justify left)
-				(hide yes)
-			)
-		)
-		(property "Footprint" "djStandard:SAMTEC-T1M-10-F-SH-L"
-			(at 12.7 86.36 0)
-			(effects
-				(font
-					(size 1.27 1.27)
-				)
-				(justify left)
-				(hide yes)
-			)
-		)
-		(property "Datasheet" "~"
-			(at 12.7 91.44 0)
-			(effects
-				(font
-					(size 1.27 1.27)
-				)
-				(justify left)
-				(hide yes)
-			)
-		)
-		(property "Description" "JANOS-STACK-DEBUG-V1"
-			(at 26.67 91.694 0)
-			(effects
-				(font
-					(size 1.27 1.27)
-				)
-				(hide yes)
-			)
-		)
-		(pin "4"
-		)
-		(pin "S2"
-		)
-		(pin "9"
-		)
-		(pin "6"
-		)
-		(pin "1"
-		)
-		(pin "10"
-		)
-		(pin "5"
-		)
-		(pin "8"
-		)
-		(pin "3"
-		)
-		(pin "S1"
-		)
-		(pin "2"
-		)
-		(pin "7"
-		)
-		(instances
-			(project ""
-				(path "/5d8326d9-7250-4cff-bfdd-e7d4c45b57a3/59a7b51e-c161-44ef-b032-7259be2f4b67"
-					(reference "J3")
-					(unit 1)
-				)
