File: components/tools/hermetica-esc-monitor/hermetica-esc-monitor.kicad_pcb (KiCad board)
At the start: 4 copper layers, 67.3 x 83.8 mm, 85 parts, among them IC1 TI-LP5912Q3.3, IC2 STM-USBLC6-2P6, J1 Conn_01x01, J10 Conn_01x01, J11 Conn_01x01, J12 Conn_01x01, J13 Conn_01x01, J14 CONNECTOR-DEBUG-SPECIFIC-ARM, J15 045138008100858+, J16 Screw_Terminal_01x03, J17 JANOS-STACK-CAN, J18 GCT-USB3075-30-A, J19 Screw_Terminal_01x03, J2 Conn_01x01, J3 Conn_01x01, J4 Conn_01x01, J5 Conn_01x01, J6 DRONE-SERVO-HEADER, J7 DRONE-SERVO-HEADER, J8 Conn_01x01, J9 Conn_01x01, U1 TPS22917DBV, U2 MB85RS1MT, U3 TI-LMR51606, U4 PESD2CANFD24V-QCZ, U5 PESD2CANFD24V-QCZ, Y1 ABRACON-ABM10AIG-48.000MHZ-4Z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

Commit message: FCU V2 REV1
Parts:
- removed IC2: STM-USBLC6-2P6, djStandard:STM-USBLC6-2P6
- removed J17: JANOS-STACK-CAN, djStandard:SAMTEC-T1M-04-F-SH-L
- removed J18: GCT-USB3075-30-A, djStandard:GCT-USB3075-30-A
- removed R29, R30: 22R, djStandard:R_0201_0603Metric
- added C18: 2.2uF, djStandard:C_0603_1608Metric, F.Cu at (17.4, 17.6)
- added C19: 2.2uF, djStandard:C_0603_1608Metric, F.Cu at (24.6, -1.78)
- added C20: 594pF, djStandard:C_0402_1005Metric, B.Cu at (10.5, 4.57)
- added C21: 100nF, djStandard:C_0402_1005Metric, F.Cu at (15.4, -7.62)
- added C22: 100nF, djStandard:C_0402_1005Metric, F.Cu at (24.1, 4.83)
- added C23: 100nF, djStandard:C_0402_1005Metric, F.Cu at (22.7, -4.70)
- added C24: 100nF, djStandard:C_0402_1005Metric, F.Cu at (24.1, 10.5)
- added C25: 100nF, djStandard:C_0402_1005Metric, F.Cu at (-1.27, -0.76)
- added C26: 100nF, djStandard:C_0402_1005Metric, F.Cu at (3.05, -7.62)
- added C27: 100nF, djStandard:C_0402_1005Metric, F.Cu at (-1.27, 4.95)
- J15: moved to B.Cu
- R10: value 1K -> 2K2
- R9: value 1K -> 1K5
- U4: moved to F.Cu
- moved R28 100.7 mm to (7.44, 6.33), turned to 90 degrees
- moved U1 96.2 mm to (9.91, 6.86), turned to 0 degrees
- moved C8 90.1 mm to (13.0, 6.84), turned to 90 degrees
- moved C17 86.2 mm to (15.1, 6.84), turned to 90 degrees
- moved U5 81.0 mm to (-23.0, 29.1), turned to -90 degrees
- moved L2 72.9 mm to (-18.9, 29.1), turned to 0 degrees
- moved U4 68.6 mm to (-23.0, 47.0), turned to -90 degrees
- moved J15 66.8 mm to (25.4, 4.45), turned to 90 degrees
- moved R17 65.5 mm to (-15.1, 28.6)
- moved R14 65.2 mm to (-15.1, 29.6), turned to 0 degrees
- moved U2 65.0 mm to (6.99, 19.8), turned to 180 degrees
- moved C5 63.2 mm to (-1.27, 2.54), turned to 180 degrees
- moved U6 59.6 mm to (-12.2, 29.1), turned to 180 degrees
- moved C3 52.5 mm to (-0.76, 12.3)
- moved J19 49.2 mm to (-29.2, 49.6), turned to -90 degrees
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Connections:
- net /BOOT0 renamed /MCU/BOOT0
- net /CLK renamed /SD-CARD/CLK
- net /CMD renamed /SD-CARD/CMD
- net /DAT0 renamed /SD-CARD/DAT0
- net /DAT1 renamed /SD-CARD/DAT1
- net /DAT2 renamed /SD-CARD/DAT2
- net /DAT3 renamed /SD-CARD/DAT3
- net /I2C2_SCL renamed /MCU/I2C2_SCL
- net /I2C2_SDA renamed /MCU/I2C2_SDA
- net /LED_GREEN renamed /MCU/LED_GREEN
- net /LED_RED renamed /MCU/LED_RED
- net /OSC+ renamed /MCU/OSC+
- net /OSC- renamed /MCU/OSC-
- net /OSC32+ renamed /MCU/OSC32+
- net /OSC32- renamed /MCU/OSC32-
- net /PDR_ON renamed /MCU/PDR_ON
- net /RESET renamed /MCU/RESET
- net /SDMMC1_CLK renamed SDMMC1_CLK
- net /SDMMC1_CMD renamed SDMMC1_CMD
- net /SDMMC1_D0 renamed SDMMC1_D0
- net /SDMMC1_D1 renamed SDMMC1_D1
- net /SDMMC1_D2 renamed SDMMC1_D2
- net /SDMMC1_D3 renamed SDMMC1_D3
- net /SDMMC1_EN renamed SDMMC1_EN
- net /SPI1_FRAM_CS renamed FRAM_CS
- net /SPI1_MISO renamed FRAM_SO
- net /SPI1_MOSI renamed FRAM_SI
- net /SPI1_SCK renamed FRAM_SCK
- net /SWCLK renamed /MCU/SWCLK
- net /SWDIO renamed /MCU/SWDIO
- net /SWO renamed /MCU/SWO
- C17 pad 1: /3V3 -> /SD-CARD/SD3V3
- C8 pad 1: /3V3 -> /SD-CARD/SD3V3
- J15 pad 4: /3V3 -> /SD-CARD/SD3V3
- J15 pad 9: unconnected-(J15-COM-Pad9) -> GND
- J15 pad CD1: unconnected-(J15-PadCD1) -> SDMMC1_CD
- MCU1 pad 100: /MCU_D- -> unconnected-(MCU1-PA11-Pad100)
- MCU1 pad 101: /MCU_D+ -> unconnected-(MCU1-PA12-Pad101)
- MCU1 pad 103: unconnected-(MCU1-VCAP-Pad103) -> /MCU/VCAP23
- MCU1 pad 105: unconnected-(MCU1-VDDLDO-Pad105) -> +3V3
- MCU1 pad 113: /FDCAN1_TX -> unconnected-(MCU1-PD1-Pad113)
- MCU1 pad 140: unconnected-(MCU1-VCAP-Pad140) -> /MCU/VCAP23
- MCU1 pad 143: unconnected-(MCU1-VDDLDO-Pad143) -> +3V3
- MCU1 pad 35: unconnected-(MCU1-VREF+-Pad35) -> /MCU/VDDA
- MCU1 pad 36: unconnected-(MCU1-VDDA-Pad36) -> /MCU/VDDA
- MCU1 pad 68: unconnected-(MCU1-VCAP-Pad68) -> /MCU/VCAP1
- MCU1 pad 70: unconnected-(MCU1-VDDLDO-Pad70) -> +3V3
- MCU1 pad 72: /FDCAN2_RX -> /MCU/FDCAN2_RX
- MCU1 pad 73: /FDCAN2_TX -> /MCU/FDCAN2_TX
- MCU1 pad 91: unconnected-(MCU1-VDD33_USB-Pad91) -> +3V3
- R23 pad 2: /3V3 -> /SD-CARD/SD3V3
- R24 pad 2: /3V3 -> /SD-CARD/SD3V3
- R25 pad 2: /3V3 -> /SD-CARD/SD3V3
- R26 pad 2: /3V3 -> /SD-CARD/SD3V3
- R27 pad 2: /3V3 -> /SD-CARD/SD3V3
- U1 pad 4: unconnected-(U1-CT-Pad4) -> /SD-CARD/TPS22917_CT
- U1 pad 5: unconnected-(U1-QOD-Pad5) -> /SD-CARD/SD3V3
- U1 pad 6: /3V3 -> /SD-CARD/SD3V3
Routing:
- net /BEC_5V: track 59.0 -> 0.00 mm, vias 1 -> 0
- net +3V3: track 4.07 -> 53.0 mm, vias 4 -> 21
- net /MCU/RESET: track 4.58 -> 44.1 mm, vias 0 -> 2
- net /SD-CARD/SD3V3: track 0.00 -> 38.7 mm, vias 0 -> 4
- net /CAN1_H: track 0.00 -> 36.5 mm
- net /CAN1_L: track 0.00 -> 36.4 mm
- net /MCU/SWO: track 0.00 -> 26.6 mm
- net /MCU/VCAP23: track 0.00 -> 22.9 mm
- net /SD-CARD/DAT2: track 1.73 -> 23.9 mm, vias 2 -> 1
- net /MCU/SWDIO: track 0.00 -> 18.9 mm
- net /SD-CARD/DAT3: track 1.73 -> 19.4 mm, vias 2 -> 1
- net /MCU/SWCLK: track 0.00 -> 14.7 mm
- net /SD-CARD/CMD: track 1.14 -> 15.0 mm
- net /USBMCU_D-: track 12.3 -> 0.00 mm
- net /SD-CARD/CLK: track 1.73 -> 13.6 mm, vias 2 -> 1
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