File: components/tools/hermetica-esc-monitor/hermetica-esc-monitor.kicad_sch (KiCad schematic)
At the start: 85 parts, among them IC1 TI-LP5912Q3.3, IC2 STM-USBLC6-2P6, J1 Conn_01x01, J10 Conn_01x01, J11 Conn_01x01, J12 Conn_01x01, J13 Conn_01x01, J14 CONNECTOR-DEBUG-SPECIFIC-ARM, J15 045138008100858+, J16 Screw_Terminal_01x03, J17 JANOS-STACK-CAN, J18 GCT-USB3075-30-A, J19 Screw_Terminal_01x03, J2 Conn_01x01, J3 Conn_01x01, J4 Conn_01x01, J5 Conn_01x01, J6 DRONE-SERVO-HEADER, J7 DRONE-SERVO-HEADER, J8 Conn_01x01, J9 Conn_01x01, U1 TPS22917DBV, U2 MB85RS1MT, U3 TI-LMR51606, U4 PESD2CANFD24V-QCZ, U5 PESD2CANFD24V-QCZ, Y1 ABRACON-ABM10AIG-48.000MHZ-4Z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

Commit message: FCU V2 REV1
Parts:
- removed C1: 4.7uF, djStandard:C_0402_1005Metric, symbol DJ:C
- removed C10, C2, C3, C4, C5, C6: 100nF, djStandard:C_0402_1005Metric, symbol DJ:C
- removed C17: 100nF, djStandard:C_0805_2012Metric, symbol DJ:C
- removed C7, C9: ?pF, djStandard:C_0402_1005Metric, symbol DJ:C
- removed C8: 10uF, djStandard:C_0805_2012Metric, symbol DJ:C
- removed IC2: STM-USBLC6-2P6, djStandard:STM-USBLC6-2P6, symbol DJ:STM-USBLC6-2P6
- removed J14: CONNECTOR-DEBUG-SPECIFIC-ARM, djStandard:PinHeader_2x05_P1.27mm_Vertical_SMD, symbol DJ:CONNECTOR-DEBUG-SPECIFIC-ARM
- removed J15: 045138008100858+, djStandard:KYOCERA-045138008100858, symbol DJ:045138008100858+
- removed J17: JANOS-STACK-CAN, djStandard:SAMTEC-T1M-04-F-SH-L, symbol DJ:JANOS-STACK-CAN
- removed J18: GCT-USB3075-30-A, djStandard:GCT-USB3075-30-A, symbol DJ:GCT-USB3075-30-A
- removed LED1: APHB1608CGKSURKC, djStandard:KINGBRIGHT-APHB1608CGKSURKC, symbol DJ:KINGBRIGHT-LED-0603-GREEN/RED
- removed MCU1: STM-STM32H755ZITx, djStandard:LQFP-144_20x20mm_P0.5mm, symbol DJ:STM-STM32H755ZITx
- removed R1, R18, R19, R20, R21, R22, R29, R3, R30, R4, R8: 22R, djStandard:R_0201_0603Metric, symbol DJ:R
- removed R10, R9: 1K, djStandard:R_0402_1005Metric, symbol DJ:R
- removed R2, R28, R5: 10K, djStandard:R_0201_0603Metric, symbol DJ:R
- removed R23, R24, R25, R26, R27: 47K, djStandard:R_0201_0603Metric, symbol DJ:R
- removed R6, R7: 10K, djStandard:R_0402_1005Metric, symbol DJ:R
- removed U1: TPS22917DBV, Package_TO_SOT_SMD:SOT-23-6, symbol Power_Management:TPS22917DBV
- removed U2: MB85RS1MT, djStandard:FUJITSU-MB85RC64TAPN-SON8, symbol Memory_NVRAM:MB85RS1MT
- removed Y1: ABRACON-ABM10AIG-48.000MHZ-4Z-T3, djStandard:ABRACON-ABM10AIG, symbol DJ:ABRACON-ABM10AIG-48.000MHZ-4Z-T3
Connections:
- no-connect marks 1 -> 0
Other:
- added sheet FRAM (fram.kicad_sch)
- added sheet MCU (mcu.kicad_sch)
- added sheet SD-CARD (sdcard.kicad_sch)
- moved on the sheet: C16, D1, J6, J7, L2, R14, R15, R16, R17, U4, U5, U6
